Commit message: All turret parts added to URDF, not placed yet. Also missing several meshes.

File: src/turret_description/urdf/turret/turret.xacro (robot description, xacro)
@@ -1,4 +1,5 @@
 <?xml version="1.0"?>
 <robot name="turret" xmlns:xacro="http://ros.org/wiki/xacro">
+  <!-- Define a number of dimensions using properties -->
   <property name="base_size_z" value="0.008" />
   <property name="secondary_base_size_z" value="0.047" />
@@ -6,12 +7,21 @@
   <property name="secondary_base_offset_y" value="0.0" />
   <property name="secondary_base_offset_z" value="${secondary_base_size_z/2 + base_size_z/2}" />
+  <property name="head_offset_x" value="0.0" />
+  <property name="head_offset_y" value="0.0" />
+  <property name="head_offset_z" value="0.0" />
    <!-- Include all component files -->
    <xacro:include filename="$(find turret_description)/urdf/materials.urdf.xacro" />
    <xacro:include filename="$(find turret_description)/urdf/turret/base.urdf.xacro" />
    <xacro:include filename="$(find turret_description)/urdf/turret/secondary_base.urdf.xacro"/>
+   <xacro:include filename="$(find turret_description)/urdf/turret/box_pan_tilt_head_xtion.urdf.xacro" />
    <!-- Add the base and wheels -->
    <base name="base" color="Black" base_size_z="${base_size_z}"/>
+   <!-- Attach the secondary base -->
   <secondary_base name="secondary_base" parent="base" color="Black" size_z="${secondary_base_size_z}">
      <origin xyz="${secondary_base_offset_x} ${secondary_base_offset_y} ${secondary_base_offset_z}" rpy="0 0 0" />
    </secondary_base>
+   <!-- Attach the pan and tilt head -->
+   <head name="head_base" parent="secondary_base" color="White">
+      <origin xyz="${head_offset_x} ${head_offset_y} ${head_offset_z}" rpy="0 0 ${PI}" />
+   </head>
 </robot>

Commit message: All turret parts added to URDF, not placed yet. Also missing several meshes.

File: src/turret_description/urdf/turret/turret.xacro (robot description, xacro)
@@ -1,4 +1,5 @@
 <?xml version="1.0"?>
 <robot name="turret" xmlns:xacro="http://ros.org/wiki/xacro">
+  <!-- Define a number of dimensions using properties -->
   <property name="base_size_z" value="0.008" />
   <property name="secondary_base_size_z" value="0.047" />
@@ -6,12 +7,21 @@
   <property name="secondary_base_offset_y" value="0.0" />
   <property name="secondary_base_offset_z" value="${secondary_base_size_z/2 + base_size_z/2}" />
+  <property name="head_offset_x" value="-0.025" />
+  <property name="head_offset_y" value="0.0" />
+  <property name="head_offset_z" value="0.055" />
    <!-- Include all component files -->
    <xacro:include filename="$(find turret_description)/urdf/materials.urdf.xacro" />
    <xacro:include filename="$(find turret_description)/urdf/turret/base.urdf.xacro" />
    <xacro:include filename="$(find turret_description)/urdf/turret/secondary_base.urdf.xacro"/>
+   <xacro:include filename="$(find turret_description)/urdf/turret/box_pan_tilt_head_xtion.urdf.xacro" />
    <!-- Add the base and wheels -->
    <base name="base" color="Black" base_size_z="${base_size_z}"/>
+   <!-- Attach the secondary base -->
   <secondary_base name="secondary_base" parent="base" color="Black" size_z="${secondary_base_size_z}">
      <origin xyz="${secondary_base_offset_x} ${secondary_base_offset_y} ${secondary_base_offset_z}" rpy="0 0 0" />
    </secondary_base>
+   <!-- Attach the pan and tilt head -->
+   <head name="head_base" parent="secondary_base" color="White">
+      <origin xyz="${head_offset_x} ${head_offset_y} ${head_offset_z}" rpy="0 0 0" />
+   </head>
 </robot>
