Commit message: Fixed bad commit.

File: src/turret_description/urdf/turret/box_pan_tilt_head_xtion.urdf.xacro (robot description, xacro)
@@ -37,9 +37,5 @@
     <!-- head pan -->
     <dynamixel_AX12_fixed parent="head_base" name="head_pan_servo">
-<<<<<<< HEAD
-       <origin xyz="0.012 0 ${-AX12_WIDTH/2}" rpy="${PI/2} 0 ${PI/2}"/>
-=======
        <origin xyz="-0.012 0 ${-AX12_WIDTH/2}" rpy="${PI/2} 0 ${-PI/2}"/>
->>>>>>> 44af0d3ee883ae7056cd3d7cbd676a79f9b89d33
     </dynamixel_AX12_fixed>
     <bioloid_F3_head_revolute parent="head_pan_servo" name="head_pan_bracket" joint_name="head_pan" ulimit="2.9" llimit="-2.9" vlimit="1.571" color="${color}">
@@ -49,9 +45,5 @@
     <!--head tilt -->
     <dynamixel_AX12_fixed parent="head_pan_bracket" name="head_tilt_servo">
-<<<<<<< HEAD
-       <origin xyz="0 0 -0.031" rpy="0 ${PI} ${PI}"/>
-=======
        <origin xyz="0 0 -0.031" rpy="0 ${PI} 0"/>
->>>>>>> 44af0d3ee883ae7056cd3d7cbd676a79f9b89d33
     </dynamixel_AX12_fixed>
     <bioloid_F2_head_revolute parent="head_tilt_servo" name="head_tilt_bracket" joint_name="head_tilt" ulimit="2.9" llimit="-2.9" vlimit="1.571" color="${color}" >
@@ -61,9 +53,5 @@
    <!-- Attach the camera -->
    <camera name="camera" parent="head_tilt_bracket" color="Black">
-<<<<<<< HEAD
-      <origin xyz="${camera_offset_x} ${camera_offset_y} ${camera_offset_z}" rpy="0 0 ${PI}" />
-=======
       <origin xyz="${camera_offset_x} ${camera_offset_y} ${camera_offset_z}" rpy="0 0 0" />
->>>>>>> 44af0d3ee883ae7056cd3d7cbd676a79f9b89d33
    </camera>
  </macro>

File: src/turret_description/urdf/turret/dynamixel_box_head_hardware.xacro (robot description, xacro)
@@ -32,8 +32,5 @@
         <origin xyz="0 0 0 " rpy="0 0 0" />
         <geometry>
-<<<<<<< HEAD
           <!--<mesh filename="package://turret_description/meshes/F3.stl" scale="${DYNAMIXEL_MESH_SCALE} ${DYNAMIXEL_MESH_SCALE} ${DYNAMIXEL_MESH_SCALE}"/>-->
-=======
->>>>>>> 44af0d3ee883ae7056cd3d7cbd676a79f9b89d33
           <box size="${F3_HEIGHT} ${F3_WIDTH} ${F3_DEPTH}"/>
         </geometry>
@@ -65,8 +62,5 @@
         <origin xyz="0 0 0" rpy="0 0 0" />
         <geometry>
-<<<<<<< HEAD
           <!--<mesh filename="package://turret_description/meshes/ax12.stl" scale="${DYNAMIXEL_MESH_SCALE} ${DYNAMIXEL_MESH_SCALE} ${DYNAMIXEL_MESH_SCALE}"/>-->
-=======
->>>>>>> 44af0d3ee883ae7056cd3d7cbd676a79f9b89d33
           <box size="${AX12_HEIGHT} ${AX12_WIDTH} ${AX12_DEPTH}"/>
         </geometry>
@@ -100,8 +94,5 @@
         <origin xyz="0 0 0 " rpy="0 0 0" />
         <geometry>
-<<<<<<< HEAD
           <!--<mesh filename="package://turret_description/meshes/F3.stl" scale="${DYNAMIXEL_MESH_SCALE} ${DYNAMIXEL_MESH_SCALE} ${DYNAMIXEL_MESH_SCALE}"/>-->
-=======
->>>>>>> 44af0d3ee883ae7056cd3d7cbd676a79f9b89d33
            <box size="${F3_DEPTH} ${F3_WIDTH} ${F3_HEIGHT}"/>
         </geometry>
@@ -135,8 +126,5 @@
         <origin xyz="0 0 0 " rpy="0 0 0" />
         <geometry>
-<<<<<<< HEAD
           <!--<mesh filename="package://turret_description/meshes/F2.stl" scale="${DYNAMIXEL_MESH_SCALE} ${DYNAMIXEL_MESH_SCALE} ${DYNAMIXEL_MESH_SCALE}"/>-->
-=======
->>>>>>> 44af0d3ee883ae7056cd3d7cbd676a79f9b89d33
           <box size="${F2_DEPTH} ${F2_HEIGHT} ${F2_WIDTH}"/>
         </geometry>

File: src/turret_description/urdf/turret/turret.xacro (robot description, xacro)
@@ -7,13 +7,7 @@
   <property name="secondary_base_offset_y" value="0.0" />
   <property name="secondary_base_offset_z" value="${secondary_base_size_z/2 + base_size_z/2}" />
-<<<<<<< HEAD
   <property name="head_offset_x" value="-0.025" />
   <property name="head_offset_y" value="0.0" />
   <property name="head_offset_z" value="0.055" />
-=======
-  <property name="head_offset_x" value="0.0" />
-  <property name="head_offset_y" value="0.0" />
-  <property name="head_offset_z" value="0.0" />
->>>>>>> 44af0d3ee883ae7056cd3d7cbd676a79f9b89d33
    <!-- Include all component files -->
    <xacro:include filename="$(find turret_description)/urdf/materials.urdf.xacro" />
@@ -29,9 +23,5 @@
    <!-- Attach the pan and tilt head -->
    <head name="head_base" parent="secondary_base" color="White">
-<<<<<<< HEAD
-      <origin xyz="${head_offset_x} ${head_offset_y} ${head_offset_z}" rpy="0 0 0" />
-=======
       <origin xyz="${head_offset_x} ${head_offset_y} ${head_offset_z}" rpy="0 0 ${PI}" />
->>>>>>> 44af0d3ee883ae7056cd3d7cbd676a79f9b89d33
    </head>
 </robot>

File: src/turret_description/urdf/turret/xtion_box.urdf.xacro (robot description, xacro)
@@ -61,9 +61,6 @@
       <link name="${name}_link">
          <visual>
-<<<<<<< HEAD
-            <origin xyz="0 0 -0.02" rpy="0 0 0" />
-=======
+            <!--<origin xyz="0 0 -0.02" rpy="0 0 0" />-->
             <origin xyz="0 0 0" rpy="0 0 0" />
->>>>>>> 44af0d3ee883ae7056cd3d7cbd676a79f9b89d33
             <geometry>
                <mesh filename="package://turret_description/meshes/xtion.stl" scale="${camera_mesh_scale} ${camera_mesh_scale} ${camera_mesh_scale}" />
